File: NodeMcuLiPolyBackpack.sch (KiCad schematic (older format))
At the start: 14 parts, among them P1 Switch, P2 G BAT, P3 Battery, P4 G 5V, U1 MCP73831

Commit message: Logo, reacomodo  v1.0
Connections:
- net VBat: now also P1.1 (P1), P2.1 (P1)
Changed lines of the file:
@@
 Rev "v1.0"
 Comp "The Inventor's House"
-Comment1 ""
+Comment1 "Xhábas"
 Comment2 ""
 Comment3 ""
@@
 $EndComp
 Wire Wire Line
-	3550 1750 4150 1750
-Wire Wire Line
-	3450 1750 2950 1750
+	2950 1750 4150 1750
 Text Label 2950 1750 0    60   ~ 0
 VBat
@@
 Wire Wire Line
 	5600 1950 5600 2150
+Wire Wire Line
+	3450 1800 3450 1750
+Connection ~ 3450 1750
+Connection ~ 3550 1750
 $EndSCHEMATC
