File: NodeMcuLiPolyBackpack.sch (KiCad schematic (older format))
At the start: 14 parts, among them P1 Switch, P2 G BAT, P3 Battery, P4 G 5V, U1 MCP73831

Commit message: Fix size
Other:
- note added: "10K = 100mA\n5K = 200mA\n2K = 500mA\n1K = 1000mA"
Changed lines of the file:
@@
 83 46 ED 50 78 11 8D BA EE CA 77 80 15 78 AC D0 25 5A 4D 41 3A 09 61 77 0A 65 03 71 3D 4E D7 4A
 20 07 E3 DA BD B3 4F 76 B6 BB 1E C2 10 5B 71 A9 1E 59 7E 31 FD 3F 66 00 F0 54 6D 0D C4 0C 00 00
-00 00 49 45 4E 44 AE 42 60 82 00
+00 00 49 45 4E 44 AE 42 60 82 06
 EndData
 $EndBitmap
+Text Notes 5500 4300 0    60   ~ 0
+10K = 100mA\n5K = 200mA\n2K = 500mA\n1K = 1000mA
 $EndSCHEMATC

Commit message: Fixes
Parts:
- added D3: MBR120, Diodes_SMD:SOD-123, symbol D_Schottky
Connections:
- net VBat: now also D3.2 (A); no longer P1.1 (P1), P1.2 (P2), P2.1 (P1)
- new net: D3.1 (K), P1.1 (P1), P1.2 (P2), P2.1 (P1)
Changed lines of the file:
@@
 Sheet 1 1
 Title "Node Mcu v3 LiPoly/LiIon Backpack"
-Date "2015-11-01"
-Rev "v1.0"
+Date "2015-12-30"
+Rev "v1.1 Rev.B"
 Comp "The Inventor's House"
 Comment1 "Andrés Sabas"
@@
 	1    0    0    -1
 $EndComp
-Wire Wire Line
-	3000 2750 4550 2750
-Wire Wire Line
-	3000 2400 3000 3050
 $Comp
 L LED D2
@@
 	1    0    0    -1
 $EndComp
-Wire Wire Line
-	5350 2750 6900 2750
-Wire Wire Line
-	6550 2450 6550 2950
-Connection ~ 6550 2750
-Wire Wire Line
-	4300 2950 4550 2950
-Wire Wire Line
-	4000 2950 3850 2950
-Wire Wire Line
-	4300 3300 4400 3300
-Wire Wire Line
-	4400 3300 4400 2950
-Connection ~ 4400 2950
-Wire Wire Line
-	3450 2950 3350 2950
-Wire Wire Line
-	3350 2950 3350 2750
-Connection ~ 3350 2750
-Wire Wire Line
-	3850 3300 4000 3300
 $Comp
 L GND #PWR01
@@
 	1    0    0    -1
 $EndComp
-Wire Wire Line
-	6550 3250 6550 3500
 $Comp
 L GND #PWR03
@@
 	1    0    0    -1
 $EndComp
-Wire Wire Line
-	6900 2850 6850 2850
-Wire Wire Line
-	6850 2850 6850 3500
-Wire Wire Line
-	6250 2850 6150 2850
-Wire Wire Line
-	5350 2850 5850 2850
-Connection ~ 5750 2850
 $Comp
 L GND #PWR05
@@
 	1    0    0    -1
 $EndComp
-Wire Wire Line
-	3000 3350 3000 3650
 $Comp
 L GND #PWR06
@@
 	1    0    0    -1
 $EndComp
-Wire Wire Line
-	2950 1750 4150 1750
-Text Label 2950 1750 0    60   ~ 0
+Text Label 2850 1750 0    60   ~ 0
 VBat
 Text Label 6550 2450 0    60   ~ 0
 VBat
-Connection ~ 3000 2750
 Text Label 5250 2150 0    60   ~ 0
 VBUS
 Text Label 3000 2400 0    60   ~ 0
 VBUS
-Wire Wire Line
-	5350 2950 5450 2950
-Wire Wire Line
-	5450 2950 5450 3900
-Wire Wire Line
-	3450 3300 3450 3600
-Wire Wire Line
-	4150 1850 3950 1850
-Wire Wire Line
-	3950 1850 3950 2150
 $Comp
 L CONN_01X02 P2
@@
 	1    0    0    -1
 $EndComp
-Wire Wire Line
-	5250 1850 5250 2150
 $Comp
 L Solder_jumper SJ1
@@
 	1    0    0    -1
 $EndComp
-Wire Wire Line
-	5750 2900 5750 2850
-Wire Wire Line
-	5750 3450 5750 3650
-Wire Wire Line
-	5750 3650 5850 3650
-Wire Wire Line
-	6250 2850 6250 4000
-Wire Wire Line
-	6150 3650 6250 3650
-Connection ~ 6250 3650
-Wire Wire Line
-	5450 3900 6250 3900
-Connection ~ 6250 3900
 $Comp
 L CONN_01X02 P4
@@
 	1    0    0    -1
 $EndComp
-Wire Wire Line
-	5250 1850 5650 1850
 $Comp
 L GND #PWR07
@@
 	1    0    0    -1
 $EndComp
-Wire Wire Line
-	5650 1950 5600 1950
-Wire Wire Line
-	5600 1950 5600 2150
-Wire Wire Line
-	3450 1800 3450 1750
-Connection ~ 3450 1750
-Connection ~ 3550 1750
 $Bitmap
 Pos 10600 6850
@@
 83 46 ED 50 78 11 8D BA EE CA 77 80 15 78 AC D0 25 5A 4D 41 3A 09 61 77 0A 65 03 71 3D 4E D7 4A
 20 07 E3 DA BD B3 4F 76 B6 BB 1E C2 10 5B 71 A9 1E 59 7E 31 FD 3F 66 00 F0 54 6D 0D C4 0C 00 00
-00 00 49 45 4E 44 AE 42 60 82 06
+00 00 49 45 4E 44 AE 42 60 82 00
 EndData
 $EndBitmap
 Text Notes 5500 4300 0    60   ~ 0
 10K = 100mA\n5K = 200mA\n2K = 500mA\n1K = 1000mA
+Wire Wire Line
+	3000 2750 4550 2750
+Wire Wire Line
+	3000 2400 3000 3050
+Wire Wire Line
+	5350 2750 6900 2750
+Wire Wire Line
+	6550 2450 6550 2950
+Connection ~ 6550 2750
+Wire Wire Line
+	4300 2950 4550 2950
+Wire Wire Line
+	4000 2950 3850 2950
+Wire Wire Line
+	4300 3300 4400 3300
+Wire Wire Line
+	4400 3300 4400 2950
+Connection ~ 4400 2950
+Wire Wire Line
+	3450 2950 3350 2950
+Wire Wire Line
+	3350 2950 3350 2750
+Connection ~ 3350 2750
+Wire Wire Line
+	3850 3300 4000 3300
+Wire Wire Line
+	6550 3250 6550 3500
+Wire Wire Line
+	6900 2850 6850 2850
+Wire Wire Line
+	6850 2850 6850 3500
+Wire Wire Line
+	6250 2850 6150 2850
+Wire Wire Line
+	5350 2850 5850 2850
+Connection ~ 5750 2850
+Wire Wire Line
+	3000 3350 3000 3650
+Connection ~ 3000 2750
+Wire Wire Line
+	5350 2950 5450 2950
+Wire Wire Line
+	5450 2950 5450 3900
+Wire Wire Line
+	3450 3300 3450 3600
+Wire Wire Line
+	4150 1850 3950 1850
+Wire Wire Line
+	3950 1850 3950 2150
+Wire Wire Line
+	5250 1850 5250 2150
+Wire Wire Line
+	5750 2900 5750 2850
+Wire Wire Line
+	5750 3450 5750 3650
+Wire Wire Line
+	5750 3650 5850 3650
+Wire Wire Line
+	6250 2850 6250 4000
+Wire Wire Line
+	6150 3650 6250 3650
+Connection ~ 6250 3650
+Wire Wire Line
+	5450 3900 6250 3900
+Connection ~ 6250 3900
+Wire Wire Line
+	5250 1850 5650 1850
+Wire Wire Line
+	5650 1950 5600 1950
+Wire Wire Line
+	5600 1950 5600 2150
+Wire Wire Line
+	3450 1800 3450 1750
+Connection ~ 3450 1750
+Connection ~ 3550 1750
+Wire Wire Line
+	2850 1750 3050 1750
+Wire Wire Line
+	3350 1750 4150 1750
+$Comp
+L D_Schottky D3
+U 1 1 56843AC2
+P 3200 1750
+F 0 "D3" H 3200 1850 50  0000 C CNN
+F 1 "MBR120" H 3200 1650 50  0000 C CNN
+F 2 "Diodes_SMD:SOD-123" H 3200 1750 60  0001 C CNN
+F 3 "" H 3200 1750 60  0000 C CNN
+	1    3200 1750
+	-1   0    0    1
+$EndComp
 $EndSCHEMATC
