File: NodeMcuLiPolyBackpack.kicad_pcb (KiCad board)
At the start: 2 copper layers, 19.8 x 26.7 mm, 15 parts, among them P1 Switch, P2 G BAT, P3 Battery, P4 G 5V, U1 MCP73831

Commit message: Fix size
Parts:
- moved P2 0.51 mm to (139.8, 97.8)
Other:
- board size 19.8 x 26.7 mm -> 19.8 x 26 mm

Commit message: Fixes
Parts:
- added D3: MBR120, Diodes_SMD:SOD-123, F.Cu at (135.4, 101.0)
Connections:
- P1 pad 1: /VBat -> Net-(D3-Pad1)
- P1 pad 2: /VBat -> Net-(D3-Pad1)
- P2 pad 1: /VBat -> Net-(D3-Pad1)
Routing:
- net Net-(D3-Pad1): track 0.00 -> 20.4 mm
- net /VBat: track 43.8 -> 23.4 mm
- net GND: track 0.07 -> 19.4 mm
- removed copper zone on F.Cu, net GND
Other:
- board size 19.8 x 26 mm -> 19.8 x 26.2 mm
- board text added: "Rev. B"
